File: RoundRobinMatrix/KiCad/RounRobin.sch (KiCad schematic (older format))
At the start: 17 parts, among them SW1 SW_Push, SW12 SW_Push, SW13 SW_Push, SW21 SW_Push, SW23 SW_Push, SW31 SW_Push, SW32 SW_Push, U1 ProMicro_r

Commit message: Update ゴースト対策について説明を追記。また回路図を説明に合わせて変更。
Parts:
- removed D1, D2, D3: D, symbol Device:D
- added D11, D22, D33: D, symbol Device:D
- renumbered SW1 to R_SW_1
Connections:
- net PIN1: now also D11.2 (A)
- net PIN2: now also D22.2 (A)
- net PIN3: now also D33.2 (A)
- net at SW12.1, SW13.1: now also D11.1 (K)
- net at SW21.1, SW23.1: now also D22.1 (K)
- net at SW31.1: now also D31.2 (A); no longer SW32.1
- net at SW31.2: now also SW32.1, D33.1 (K); no longer D31.2 (A)
